File: schematics/rfid board v2/rfid board v2.sch (KiCad schematic (older format))
At the start: 17 parts, among them J1 RFID_RJ45, J2 CONN_15, J3 CONN_15, J5 POWER_JACK, J6 CONN_02, K1 SANYOU_SRD_Form_C, Q1 TRANS_NPN-P2N2222A, U1 VREG_3V3

Commit message: Updated components to match new libaries
Parts:
- D1, D3: symbol D -> Device:D
- D2: symbol D_Schottky -> Device:D_Schottky
- F1: symbol FUSE -> rfid-board-v2-rescue:FUSE
- J1: symbol RJ45_Shielded -> Connector:RJ45_Shielded
- J2, J3: symbol CONN_15 -> SparkFun-Connectors:CONN_15
- J5: symbol POWER_JACK -> SparkFun-Connectors:POWER_JACK
- J6: symbol CONN_02 -> SparkFun-Connectors:CONN_02
- K1: symbol SANYOU_SRD_Form_C -> rfid-board-v2-rescue:SANYOU_SRD_Form_C
- MH1, MH2, MH3: symbol MountingHole -> Mechanical:MountingHole
- Q1: symbol TRANS_NPN-P2N2222A -> SparkFun-DiscreteSemi:TRANS_NPN-P2N2222A
- R1: symbol 1KOHM-HORIZ-1_4W-5% -> SparkFun-Resistors:1KOHM-HORIZ-1_4W-5%
- R2: symbol 10KOHM-HORIZ-1_4W-5% -> SparkFun-Resistors:10KOHM-HORIZ-1_4W-5%
- U1: symbol VREG_3V3 -> smart_classroom_components:VREG_3V3
